Commit message: urdf file fixed physics and gravity enabled

File: trunk/kraken/scenes/kraken_stripped.urdf (robot description, URDF)
Before this commit: robot kraken, 7 links, 6 joints
Links:
- link base_link: geometry collision mesh filename=package://UWSim/kraken/robot/new_model_kraken.3ds; visual mesh filename=package://UWSim/kraken/robot/new_model_kraken.3ds

Commit message: Everyrhing fixed in environment

File: trunk/kraken/scenes/kraken_stripped.urdf (robot description, URDF)
Before this commit: robot kraken, 7 links, 6 joints
Links:
- added link camera_bottom_optical
- added link camera_front_optical
- added link depth_sensor
- added link imu_link
- link base_link: mass 35 -> None
Joints:
- added joint camera_bottom_optical_to_base_link: type fixed, parent camera_bottom, child camera_bottom_optical, origin xyz=0 0.0 0 rpy=0 0 -1.57, axis 0 0 1
- added joint camera_front_optical_to_base_link: type fixed, parent camera_front, child camera_front_optical, origin xyz=0 0.0 0 rpy=0 0 -1.57, axis 0 0 1
- added joint depth_sensor_to_base_link: type fixed, parent base_link, child depth_sensor, origin xyz=-0.302 0.00 -0.03 rpy=0 0 0, axis 0 0 1
- added joint imu_to_base_link: type fixed, parent base_link, child imu_link, origin xyz=-0.602 0.00 -0.03 rpy=0 0 0, axis 0 0 1
- joint camera_bottom_to_base_link: origin xyz=0.05 -0.0 -0.03 rpy=0 0 0 -> xyz=0.05 -0.0 0.03 rpy=0 3.14 0
- joint camera_front_to_base_link: origin xyz=0.358 -0.0 0.13 rpy=0 -1.57 0 -> xyz=0.358 -0.0 -0.13 rpy=0 -1.57 0
- joint left_heave_thruster_to_base_link: origin xyz=-0.0 0.17 0.06 rpy=0 0.0 0 -> xyz=-0.0 0.17 -0.06 rpy=0 0.0 0
- joint left_surge_thruster_to_base_link: origin xyz=-0.452 0.17 0.00 rpy=0 0.0 0 -> xyz=-0.452 0.17 -0.01 rpy=0 0.0 0
- joint right_heave_thruster_to_base_link: origin xyz=-0.0 -0.17 0.06 rpy=0 0.0 0 -> xyz=-0.0 -0.17 -0.06 rpy=0 0.0 0
- joint right_surge_thruster_to_base_link: origin xyz=-0.452 -0.17 0.00 rpy=0 0.0 0 -> xyz=-0.452 -0.17 -0.01 rpy=0 0.0 0

File: trunk/kraken/scenes/objects/pool.urdf.xacro (robot description, xacro)
@@ -17,5 +17,5 @@
   		xmlns:physics="http://playerstage.sourceforge.net/gazebo/xmlschema/#physics"
        	xmlns:xacro="http://www.ros.org/wiki/xacro">
-	<xacro:macro name="pool">
+	<xacro:macro name="pool" params="*origin">
 	  <link name="pool">
         <visual>
@@ -23,5 +23,5 @@
 		    <mesh filename="package://UWSim/kraken/terrain/pool.osg"/>
   		  </geometry>
-  		  <origin rpy="0 3.14 0" xyz="0 0 0"/>
+  		  <insert_block name="origin" />
   	    </visual>
         <collision>
@@ -29,5 +29,5 @@
 		    <mesh filename="package://UWSim/kraken/terrain/pool.osg"/>
   		  </geometry>
-  		  <origin rpy="0 0 0" xyz="0 0 0"/>
+  		  <insert_block name="origin" />
         </collision>
       </link>

File: trunk/kraken/scenes/scene.urdf (robot description, URDF)
Before this commit: robot scene, 8 links, 7 joints
Joints:
- joint gate_marker_to_pool: origin xyz=2 2 0 rpy=0 0 0.0 -> xyz=0 0 0 rpy=0 0 0.0

File: trunk/kraken/scenes/test.urdf.xacro (robot description, xacro)
@@ -26,7 +26,9 @@
   <include filename="$(find UWSim)/kraken/scenes/objects/pool.urdf.xacro"/>
   <include filename="$(find UWSim)/kraken/scenes/objects/L_rod.urdf.xacro"/>
-  <xacro:pool />
+  <xacro:pool >
+    <origin xyz="0 0 0" rpy="0 0 0.0" />
+  </xacro:pool>
   <xacro:marker position = "gate" parent = "pool">
-    <origin xyz="2 2 0" rpy="0 0 0.0" />
+    <origin xyz="0 0 0" rpy="0 0 0.0" />
   </xacro:marker>
   <xacro:buoy_blue position = "gate" parent = "pool">
